File: GitHub_Board.kicad_pcb (KiCad board)
At the start: 6 copper layers, 87 parts, among them J1 Conn_02x10_Top_Bottom, J2 Conn_02x10_Top_Bottom, J3 Conn_02x10_Top_Bottom, J4 Conn_01x05, J5 Conn_01x05, J6 Conn_01x05

Commit message: Finished PDB.
Parts:
- moved C1 80.2 mm to (229.3, 189.0), turned to 180 degrees
- moved H16 54.6 mm to (184.0, 159.5)
- moved H12 42.0 mm to (184.0, 201.5)
- moved H4 42.0 mm to (181.0, 222.5)
- moved H5 41.0 mm to (223.0, 222.5)
- moved H8 35.0 mm to (220.0, 201.5)
- moved H9 2.24 mm to (181.0, 258.5)
- moved H2 2.00 mm to (223.0, 258.5)
- moved H1 1.41 mm to (181.0, 101.5)
- moved J4 1.34 mm to (239.7, 108.9)
- moved J5 1.31 mm to (167.8, 251.7)
- moved J6 1.30 mm to (190.8, 146.8)
- moved H17 1.00 mm to (223.0, 101.5)
- moved H6 1.00 mm to (181.0, 137.5)
Routing:
- net GND: track 723.5 -> 2.05 mm, vias 1 -> 0
- net +12V: track 322.9 -> 0.14 mm
- net Net-(PI1-Pin_1): track 93.6 -> 16.6 mm, vias 1 -> 0
- net /EN6-: track 286.4 -> 277.6 mm, vias 0 -> 1
- net +5V: track 90.5 -> 94.5 mm, vias 0 -> 4
- net /EN6+: track 279.5 -> 277.0 mm, vias 0 -> 1
- net /LS4: track 279.8 -> 281.2 mm
- net /LS6: track 290.5 -> 289.5 mm, vias 3 -> 4
- net /LS2: track 340.5 -> 339.7 mm, vias 4 -> 5
- net /LS5: track 290.4 -> 291.3 mm, vias 3 -> 4
- net /LS1: track 345.0 -> 345.6 mm, vias 4 -> 5
- net /XT305-: vias 0 -> 2
- net Net-(J3-Pin_1): vias 4 -> 2
- net /XT306-: vias 0 -> 2
- net /XT306+: vias 0 -> 2
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Other:
- board outline added: 304.8 x 165.1 mm
